File: 542xISA.kicad_pcb (KiCad board)
At the start: 2 copper layers, 163.6 x 83.4 mm, 101 parts, among them J1 Conn_02x13_Odd_Even, J2 0, J3 0, P1 VGA-PORT, U1 GD5428, U11 KM416C256, U12 KM416C256, U13 KM416C256, U14 KM416C256, U2 LM334M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

Commit message: final version
Parts:
- removed RP1, RP2, RP3: 33, Resistor_SMD:R_Array_Concave_4x0603
- added C7: 100n, Capacitor_SMD:C_0805_2012Metric, B.Cu at (192.8, 122.6)
- added RN1: 33, Resistor_SMD:R_Array_Convex_8x0602, F.Cu at (159.0, 111.5)
- added RN2: 33, Resistor_SMD:R_Array_Concave_4x0603, F.Cu at (158.9, 107.2)
- C20: moved to B.Cu
- R7: footprint Resistor_SMD:R_1206_3216Metric_Pad1.30x1.75mm_HandSolder -> Resistor_SMD:R_0805_2012Metric
- moved R10 32.5 mm to (141.9, 93.6), turned to 0 degrees
- moved R9 25.7 mm to (141.9, 91.7), turned to 0 degrees
- moved R73 11.9 mm to (104.9, 91.1)
- moved C34 10.8 mm to (243.8, 127.9), turned to -90 degrees
- moved R69 7.92 mm to (104.9, 89.2)
- moved C13 7.03 mm to (152.6, 128.2)
- moved R63 6.24 mm to (104.8, 85.2)
- moved C20 6.18 mm to (187.6, 92.5), turned to -90 degrees
- moved R61 6.11 mm to (104.8, 83.3)
- moved R59 6.10 mm to (104.8, 81.4)
- moved R57 5.84 mm to (104.8, 79.5)
- moved R55 5.71 mm to (104.8, 77.6)
- moved R7 5.60 mm to (151.4, 107.1), turned to 90 degrees
- moved L1 4.72 mm to (149.9, 129.1)
- moved R8 4.71 mm to (157.6, 104.3)
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Connections:
- net IREF renamed /IREF
- net Net-(U1-AVDD1) renamed /AVDD1
- net Net-(U1-AVDD4) renamed /AVDD4
- R7 pad 1: MA4 -> CAS0
- R7 pad 2: Net-(U1-MA4) -> Net-(U1-~{CAS0})
- U1 pad 138: Net-(RP3-R1.2) -> Net-(U1-~{CAS0})
- U1 pad 149: Net-(U1-MA4) -> Net-(RN1-R5.1)
- U11 pad 10: PD7 -> PD1
- U11 pad 2: PD0 -> PD15
- U11 pad 3: PD1 -> PD13
- U11 pad 31: PD8 -> PD0
- U11 pad 32: PD9 -> PD2
- U11 pad 33: PD10 -> PD4
- U11 pad 34: PD11 -> PD6
- U11 pad 36: PD12 -> PD8
- U11 pad 37: PD13 -> PD10
- U11 pad 38: PD14 -> PD12
- U11 pad 39: PD15 -> PD14
- U11 pad 4: PD2 -> PD11
- U11 pad 5: PD3 -> PD9
- U11 pad 7: PD4 -> PD7
- U11 pad 9: PD6 -> PD3
- U12 pad 10: PD23 -> PD17
- U12 pad 2: PD16 -> PD31
- U12 pad 3: PD17 -> PD29
- U12 pad 31: PD24 -> PD16
- U12 pad 32: PD25 -> PD18
- U12 pad 33: PD26 -> PD20
- U12 pad 34: PD27 -> PD22
- U12 pad 36: PD28 -> PD24
- U12 pad 37: PD29 -> PD26
- U12 pad 38: PD30 -> PD28
- U12 pad 39: PD31 -> PD30
- U12 pad 4: PD18 -> PD27
- U12 pad 5: PD19 -> PD25
- U12 pad 7: PD20 -> PD23
- U12 pad 9: PD22 -> PD19
- U13 pad 10: PD7 -> PD1
- U13 pad 2: PD0 -> PD15
- U13 pad 3: PD1 -> PD13
- U13 pad 31: PD8 -> PD0
- U13 pad 32: PD9 -> PD2
- U13 pad 33: PD10 -> PD4
- U13 pad 34: PD11 -> PD6
- U13 pad 36: PD12 -> PD8
- U13 pad 37: PD13 -> PD10
- U13 pad 38: PD14 -> PD12
- U13 pad 39: PD15 -> PD14
- U13 pad 4: PD2 -> PD11
- U13 pad 5: PD3 -> PD9
- U13 pad 7: PD4 -> PD7
- U13 pad 9: PD6 -> PD3
- U14 pad 10: PD23 -> PD17
- U14 pad 2: PD16 -> PD31
- U14 pad 3: PD17 -> PD29
- U14 pad 31: PD24 -> PD16
- U14 pad 32: PD25 -> PD18
- U14 pad 33: PD26 -> PD20
- U14 pad 34: PD27 -> PD22
- U14 pad 36: PD28 -> PD24
- U14 pad 37: PD29 -> PD26
- U14 pad 38: PD30 -> PD28
- U14 pad 39: PD31 -> PD30
- U14 pad 4: PD18 -> PD27
- U14 pad 5: PD19 -> PD25
- U14 pad 7: PD20 -> PD23
- U14 pad 9: PD22 -> PD19
Routing:
- net MA0: track 108.6 -> 155.9 mm, vias 4 -> 6
- net CAS3: track 59.0 -> 22.1 mm
- net Net-(U1-~{CAS3}): track 2.66 -> 36.6 mm, vias 0 -> 4
- net RAS1: track 71.1 -> 104.4 mm, vias 2 -> 4
- net CAS2: track 51.6 -> 22.4 mm
- net Net-(U1-~{CAS2}): track 2.51 -> 31.0 mm
- net GND: track 177.1 -> 151.8 mm, vias 174 -> 153
- net PD15: track 60.9 -> 76.2 mm
- net PD6: track 68.4 -> 53.8 mm, vias 2 -> 0
- net PD31: track 70.2 -> 84.5 mm
- net PD18: track 71.6 -> 58.0 mm, vias 2 -> 0
- net CAS0: track 51.2 -> 38.1 mm
- net Net-(U1-~{CAS0}): track 0.00 -> 13.1 mm
- net PD4: track 65.7 -> 53.4 mm, vias 2 -> 0
- net PD16: track 68.6 -> 56.8 mm, vias 4 -> 0
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