File: 542xISA.kicad_sch (KiCad schematic)
At the start: 99 parts, among them J1 Conn_02x13_Odd_Even, J2 0, J3 0, P1 VGA-PORT, U1 GD5428, U11 KM416C256, U12 KM416C256, U13 KM416C256, U14 KM416C256, U2 LM334M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

Commit message: final version
Parts:
- removed RP1, RP2: 33, Resistor_SMD:R_Array_Concave_4x0603, symbol Device:R_Pack04
- added C7: 100n, Capacitor_SMD:C_0805_2012Metric, symbol Device:C
- added RN1: 33, Resistor_SMD:R_Array_Convex_8x0602, symbol Device:R_Pack08
- R7: footprint Resistor_SMD:R_1206_3216Metric_Pad1.30x1.75mm_HandSolder -> Resistor_SMD:R_0805_2012Metric
- renumbered RP3 to RN2
Connections:
- net CAS0: now also R7.1; no longer RN2.1 (R1.1)
- net GND: now also C7.2
- net MA0: now also RN1.16 (R1.2)
- net MA1: now also RN1.15 (R2.2)
- net MA2: now also RN1.14 (R3.2)
- net MA3: now also RN1.13 (R4.2)
- net MA4: now also RN1.12 (R5.2); no longer R7.1
- net MA5: now also RN1.11 (R6.2)
- net MA6: now also RN1.10 (R7.2)
- net MA7: now also RN1.9 (R8.2)
- net MA8: now also RN2.4 (R4.1)
- net PD0: now also U11.31 (DQ8), U13.31 (DQ8); no longer U11.2 (DQ0), U13.2 (DQ0)
- net PD1: now also U11.10 (DQ7), U13.10 (DQ7); no longer U11.3 (DQ1), U13.3 (DQ1)
- net PD10: now also U11.37 (DQ13), U13.37 (DQ13); no longer U11.33 (DQ10), U13.33 (DQ10)
- net PD11: now also U11.4 (DQ2), U13.4 (DQ2); no longer U11.34 (DQ11), U13.34 (DQ11)
- net PD12: now also U11.38 (DQ14), U13.38 (DQ14); no longer U11.36 (DQ12), U13.36 (DQ12)
- net PD13: now also U11.3 (DQ1), U13.3 (DQ1); no longer U11.37 (DQ13), U13.37 (DQ13)
- net PD14: now also U11.39 (DQ15), U13.39 (DQ15); no longer U11.38 (DQ14), U13.38 (DQ14)
- net PD15: now also U11.2 (DQ0), U13.2 (DQ0); no longer U11.39 (DQ15), U13.39 (DQ15)
- net PD16: now also U12.31 (DQ8), U14.31 (DQ8); no longer U12.2 (DQ0), U14.2 (DQ0)
- net PD17: now also U12.10 (DQ7), U14.10 (DQ7); no longer U12.3 (DQ1), U14.3 (DQ1)
- net PD18: now also U12.32 (DQ9), U14.32 (DQ9); no longer U12.4 (DQ2), U14.4 (DQ2)
- net PD19: now also U12.9 (DQ6), U14.9 (DQ6); no longer U12.5 (DQ3), U14.5 (DQ3)
- net PD2: now also U11.32 (DQ9), U13.32 (DQ9); no longer U11.4 (DQ2), U13.4 (DQ2)
- net PD20: now also U12.33 (DQ10), U14.33 (DQ10); no longer U12.7 (DQ4), U14.7 (DQ4)
- net PD22: now also U12.34 (DQ11), U14.34 (DQ11); no longer U12.9 (DQ6), U14.9 (DQ6)
- net PD23: now also U12.7 (DQ4), U14.7 (DQ4); no longer U12.10 (DQ7), U14.10 (DQ7)
- net PD24: now also U12.36 (DQ12), U14.36 (DQ12); no longer U12.31 (DQ8), U14.31 (DQ8)
- net PD25: now also U12.5 (DQ3), U14.5 (DQ3); no longer U12.32 (DQ9), U14.32 (DQ9)
- net PD26: now also U12.37 (DQ13), U14.37 (DQ13); no longer U12.33 (DQ10), U14.33 (DQ10)
- net PD27: now also U12.4 (DQ2), U14.4 (DQ2); no longer U12.34 (DQ11), U14.34 (DQ11)
- net PD28: now also U12.38 (DQ14), U14.38 (DQ14); no longer U12.36 (DQ12), U14.36 (DQ12)
- net PD29: now also U12.3 (DQ1), U14.3 (DQ1); no longer U12.37 (DQ13), U14.37 (DQ13)
- net PD3: now also U11.9 (DQ6), U13.9 (DQ6); no longer U11.5 (DQ3), U13.5 (DQ3)
- net PD30: now also U12.39 (DQ15), U14.39 (DQ15); no longer U12.38 (DQ14), U14.38 (DQ14)
- net PD31: now also U12.2 (DQ0), U14.2 (DQ0); no longer U12.39 (DQ15), U14.39 (DQ15)
- net PD4: now also U11.33 (DQ10), U13.33 (DQ10); no longer U11.7 (DQ4), U13.7 (DQ4)
- net PD6: now also U11.34 (DQ11), U13.34 (DQ11); no longer U11.9 (DQ6), U13.9 (DQ6)
- net PD7: now also U11.7 (DQ4), U13.7 (DQ4); no longer U11.10 (DQ7), U13.10 (DQ7)
- net PD8: now also U11.36 (DQ12), U13.36 (DQ12); no longer U11.31 (DQ8), U13.31 (DQ8)
- net PD9: now also U11.5 (DQ3), U13.5 (DQ3); no longer U11.32 (DQ9), U13.32 (DQ9)
- net RAS0: now also RN2.3 (R3.1); no longer RN2.4 (R4.1)
- net RAS1: now also RN2.2 (R2.1); no longer RN2.3 (R3.1)
- net VCC: now also C7.1
- net WE0: now also RN2.1 (R1.1); no longer RN2.2 (R2.1)
- net AVDD1: now reaches C16.1, C17.1, L2.2, U1.66 (AVDD1)
- net at U1.148 (MA5): now also RN1.6 (R6.1)
- net at U1.147 (MA6): now also RN1.7 (R7.1)
- net at U1.146 (MA7): now also RN1.8 (R8.1)
- net at U1.145 (MA8): now also RN2.5 (R4.2)
- net at U1.153 (MA0): now also RN1.1 (R1.1)
- net at U1.152 (MA1): now also RN1.2 (R2.1)
- net at U1.151 (MA2): now also RN1.3 (R3.1)
- net at U1.150 (MA3): now also RN1.4 (R4.1)
- net at U1.142 (~{RAS}): now also RN2.6 (R3.2); no longer RN2.5 (R4.2)
- net at U1.141 (~{OE}): now also RN2.7 (R2.2); no longer RN2.6 (R3.2)
- net at U1.139 (~{WE}): now also RN2.8 (R1.2); no longer RN2.7 (R2.2)
- net at U1.138 (~{CAS0}): now also R7.2; no longer RN2.8 (R1.2)
- net at U1.149 (MA4): now also RN1.5 (R5.1); no longer R7.2
- net AVDD4: now reaches C12.1, C13.1, L1.1, U1.154 (AVDD4)
- no-connect marks 72 -> 73
Other:
- moved on the sheet: C10, C11, C12, C13, C24, C33, C41, C42, C43, C44, C45, C46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
